File: rpipowerhat/rpipowerhat.brd (EAGLE design)
At the start: 80 x 100 mm, 4 parts, among them X1 MKDSN1,5/2-5,08, X2 MKDSN1,5/2-5,08

Commit message: add device
Parts:
- removed U$1: OKX-T3-D12, suhyouri:OKX-T3-D12
- added LED1: (no value), adafruit:CHIPLED_0603
- added R2: 1k, rcl:R0603
- added R3: 1k, suhyouri:RTRIM3296W
- added U1: OKX-T3-D12, suhyouri:OKX-T3-D12
Connections:
- new net N$1: R1.1, R3.3
- new net N$2: R1.2, U1.2
- new net N$3: LED1.C, R2.2
- net +12V: now also U1.4; no longer U$1.5
- net +5V: now also LED1.A, U1.1; no longer U$1.1
- net GND: now also R2.1, R3.2, U1.3; no longer U$1.3

Commit message: homework done
Parts:
- moved R2 50.4 mm to (5.08, 15.2)
- moved R3 48.5 mm to (20.3, 15.2)
- moved LED1 38.6 mm to (5.08, 6.35)
- moved X1 26.1 mm to (44.5, 39.4)
- moved X2 16.5 mm to (17.8, 50.8)
- moved U1 4.02 mm to (8.89, -22.9)
Changed lines of the file:
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@@
 <attribute name="VALUE" x="8.255" y="18.415" size="1.27" layer="27"/>
 </element>
-<element name="X1" library="con-phoenix-508" library_urn="urn:adsk.eagle:library:176" package="MKDSN1,5/2-5,08" package3d_urn="urn:adsk.eagle:package:9630/1" value="MKDSN1,5/2-5,08" x="25.4" y="21.59" smashed="yes">
-<attribute name="NAME" x="20.6489" y="26.035" size="1.27" layer="25"/>
-<attribute name="POPULARITY" value="14" x="25.4" y="21.59" size="1.778" layer="27" display="off"/>
-<attribute name="VALUE" x="32.385" y="17.78" size="1.27" layer="27" rot="R90"/>
+<element name="X1" library="con-phoenix-508" library_urn="urn:adsk.eagle:library:176" package="MKDSN1,5/2-5,08" package3d_urn="urn:adsk.eagle:package:9630/1" value="MKDSN1,5/2-5,08" x="44.45" y="39.37" smashed="yes">
+<attribute name="NAME" x="39.6989" y="43.815" size="1.27" layer="25"/>
+<attribute name="POPULARITY" value="14" x="44.45" y="39.37" size="1.778" layer="27" display="off"/>
+<attribute name="VALUE" x="51.435" y="35.56" size="1.27" layer="27" rot="R90"/>
 </element>
-<element name="X2" library="con-phoenix-508" library_urn="urn:adsk.eagle:library:176" package="MKDSN1,5/2-5,08" package3d_urn="urn:adsk.eagle:package:9630/1" value="MKDSN1,5/2-5,08" x="11.43" y="35.56" smashed="yes">
-<attribute name="NAME" x="6.6789" y="40.005" size="1.27" layer="25"/>
-<attribute name="POPULARITY" value="14" x="11.43" y="35.56" size="1.778" layer="27" display="off"/>
-<attribute name="VALUE" x="18.415" y="31.75" size="1.27" layer="27" rot="R90"/>
+<element name="X2" library="con-phoenix-508" library_urn="urn:adsk.eagle:library:176" package="MKDSN1,5/2-5,08" package3d_urn="urn:adsk.eagle:package:9630/1" value="MKDSN1,5/2-5,08" x="17.78" y="50.8" smashed="yes">
+<attribute name="NAME" x="13.0289" y="55.245" size="1.27" layer="25"/>
+<attribute name="POPULARITY" value="14" x="17.78" y="50.8" size="1.778" layer="27" display="off"/>
+<attribute name="VALUE" x="24.765" y="46.99" size="1.27" layer="27" rot="R90"/>
 </element>
-<element name="U1" library="suhyouri" package="OKX-T3-D12" value="OKX-T3-D12" x="5.08" y="-21.59" smashed="yes">
-<attribute name="NAME" x="1.27" y="-13.97" size="1.27" layer="25"/>
-<attribute name="VALUE" x="1.27" y="-15.24" size="1.27" layer="27"/>
+<element name="U1" library="suhyouri" package="OKX-T3-D12" value="OKX-T3-D12" x="8.89" y="-22.86" smashed="yes">
+<attribute name="NAME" x="12.7" y="-16.51" size="1.27" layer="25"/>
+<attribute name="VALUE" x="5.08" y="-16.51" size="1.27" layer="27"/>
 </element>
-<element name="R3" library="suhyouri" package="RTRIM3296W" value="1k" x="-15.24" y="-17.78" smashed="yes">
-<attribute name="NAME" x="-17.89" y="-22.28" size="1.27" layer="25" rot="R90"/>
-<attribute name="VALUE" x="-11.29" y="-22.28" size="1.27" layer="27" rot="R90"/>
+<element name="R3" library="suhyouri" package="RTRIM3296W" value="1k" x="20.32" y="15.24" smashed="yes">
+<attribute name="NAME" x="17.67" y="10.74" size="1.27" layer="25" rot="R90"/>
+<attribute name="VALUE" x="24.27" y="10.74" size="1.27" layer="27" rot="R90"/>
 </element>
-<element name="LED1" library="adafruit" package="CHIPLED_0603" value="" x="-22.86" y="-20.32" smashed="yes">
-<attribute name="NAME" x="-23.495" y="-21.59" size="1.27" layer="25" rot="R90"/>
-<attribute name="VALUE" x="-20.955" y="-21.59" size="1.27" layer="27" rot="R90"/>
+<element name="LED1" library="adafruit" package="CHIPLED_0603" value="" x="5.08" y="6.35" smashed="yes">
+<attribute name="NAME" x="4.445" y="5.08" size="1.27" layer="25" rot="R90"/>
+<attribute name="VALUE" x="6.985" y="5.08" size="1.27" layer="27" rot="R90"/>
 </element>
-<element name="R2" library="rcl" library_urn="urn:adsk.eagle:library:334" package="R0603" package3d_urn="urn:adsk.eagle:package:23555/3" value="1k" x="-22.86" y="-26.67" smashed="yes">
-<attribute name="NAME" x="-23.495" y="-26.035" size="1.27" layer="25"/>
-<attribute name="POPULARITY" value="77" x="-22.86" y="-26.67" size="1.778" layer="27" display="off"/>
-<attribute name="SPICEPREFIX" value="R" x="-22.86" y="-26.67" size="1.778" layer="27" display="off"/>
-<attribute name="VALUE" x="-23.495" y="-28.575" size="1.27" layer="27"/>
+<element name="R2" library="rcl" library_urn="urn:adsk.eagle:library:334" package="R0603" package3d_urn="urn:adsk.eagle:package:23555/3" value="1k" x="5.08" y="15.24" smashed="yes">
+<attribute name="NAME" x="4.445" y="15.875" size="1.27" layer="25"/>
+<attribute name="POPULARITY" value="77" x="5.08" y="15.24" size="1.778" layer="27" display="off"/>
+<attribute name="SPICEPREFIX" value="R" x="5.08" y="15.24" size="1.778" layer="27" display="off"/>
+<attribute name="VALUE" x="32.385" y="26.035" size="1.27" layer="27"/>
 </element>
 </elements>
@@
 <contactref element="R3" pad="2"/>
 <contactref element="R2" pad="1"/>
-<wire x1="-15.24" y1="-17.78" x2="-23.71" y2="-26.67" width="0" layer="19" extent="1-1"/>
-<wire x1="17.78" y1="-21.59" x2="-15.24" y2="-17.78" width="0" layer="19" extent="1-1"/>
-<wire x1="22.8389" y1="21.615" x2="17.78" y2="-21.59" width="0" layer="19" extent="1-1"/>
-<wire x1="8.8689" y1="35.585" x2="22.8389" y2="21.615" width="0" layer="19" extent="1-1"/>
+<wire x1="20.32" y1="15.24" x2="4.23" y2="15.24" width="0" layer="19" extent="1-1"/>
+<wire x1="21.59" y1="-22.86" x2="20.32" y2="15.24" width="0" layer="19" extent="1-1"/>
+<wire x1="41.8889" y1="39.395" x2="21.59" y2="-22.86" width="0" layer="19" extent="1-1"/>
+<wire x1="15.2189" y1="50.825" x2="41.8889" y2="39.395" width="0" layer="19" extent="1-1"/>
 </signal>
 <signal name="+12V">
 <contactref element="X1" pad="2"/>
 <contactref element="U1" pad="4"/>
-<wire x1="5.08" y1="-21.59" x2="27.9189" y2="21.615" width="0" layer="19" extent="1-1"/>
+<wire x1="8.89" y1="-22.86" x2="46.9689" y2="39.395" width="0" layer="19" extent="1-1"/>
 </signal>
 <signal name="+5V">
@@
 <contactref element="U1" pad="1"/>
 <contactref element="LED1" pad="A"/>
-<wire x1="22.86" y1="-21.59" x2="13.9489" y2="35.585" width="0" layer="19" extent="1-1"/>
-<wire x1="-22.86" y1="-21.07" x2="22.86" y2="-21.59" width="0" layer="19" extent="1-1"/>
+<wire x1="26.67" y1="-22.86" x2="20.2989" y2="50.825" width="0" layer="19" extent="1-1"/>
+<wire x1="5.08" y1="5.6" x2="26.67" y2="-22.86" width="0" layer="19" extent="1-1"/>
 </signal>
 <signal name="N$2">
 <contactref element="U1" pad="2"/>
 <contactref element="R1" pad="2"/>
-<wire x1="20.32" y1="-21.59" x2="9.74" y2="20.32" width="0" layer="19" extent="1-1"/>
+<wire x1="24.13" y1="-22.86" x2="9.74" y2="20.32" width="0" layer="19" extent="1-1"/>
 </signal>
 <signal name="N$1">
 <contactref element="R1" pad="1"/>
 <contactref element="R3" pad="3"/>
-<wire x1="8.04" y1="20.32" x2="-15.24" y2="-15.24" width="0" layer="19" extent="1-1"/>
+<wire x1="8.04" y1="20.32" x2="20.32" y2="17.78" width="0" layer="19" extent="1-1"/>
 </signal>
 <signal name="N$3">
 <contactref element="LED1" pad="C"/>
 <contactref element="R2" pad="2"/>
-<wire x1="-22.86" y1="-19.57" x2="-22.01" y2="-26.67" width="0" layer="19" extent="1-1"/>
+<wire x1="5.08" y1="7.1" x2="5.93" y2="15.24" width="0" layer="19" extent="1-1"/>
 </signal>
 </signals>
