File: rpipowerhat/rpipowerhat.sch (EAGLE design)
At the start: 4 parts, among them X1 MKDSN1,5/2-5,08, X2 MKDSN1,5/2-5,08

Commit message: add device
Parts:
- added LED1: (no value), adafruit:LEDCHIPLED_0603
- added R2: 1k, rcl:R-US_R0603
- added R3: 1k, suhyouri:POT-3296
- renumbered U$1 to U1
Connections:
- new net N$1: R1.1, R3.E
- new net N$2: R1.2, U1.TRIM
- new net N$3: LED1.C, R2.2
- net +12V: now also U1.+VIN; no longer U1.REMOTE
- net +5V: now also LED1.A
- net GND: now also R2.1, R3.S
Other:
- note added: "R trim 1.475k -> 5V output"
- note added: "input voltage range 8.3-13.8v"
- moved on the sheet: R1, X2-1, X2-2

Commit message: homework done
Other:
- moved on the sheet: LED1, R1, R2, R3, U1, X1-1, X1-2, X2-1, X2-2
